File: hardware/Apollo.kicad_pcb (KiCad board)
At the start: 2 copper layers, 101.2 x 199.1 mm, 80 parts, among them J1 TYPE-C 16PIN 2MD(073), J2 Conn_ARM_JTAG_SWD_10, J22 Conn_01x16, J3 Conn_02x03_Odd_Even, J4 Conn_02x04_Odd_Even, Q1 DMP1045U-7, Q2 SS8550, Q3 SS8050, Q4 SS8050, SW1 MK-12C01-G1.5, SW2 TS-1095PS-A1B2-C3D2, SW3 TS-1095PS-A1B2-C3D2, SW4 K1-1507SA-03, U1 TPS63031DSK, U10 PY25Q128HA, U11 SAINTCON-Minibadge, U12 SAINTCON-Minibadge, U2 RP2350A-QFN60, U3 SAINTCON-Minibadge, U4 SAINTCON-Minibadge, U5 SAINTCON-Minibadge, U6 SAINTCON-Minibadge, U7 24CS02, U8 SAINTCON-Minibadge, U9 SAINTCON-Minibadge, Y1 12Mhz

Commit message: Added achievement screen and minor edits
Parts:
- moved U5 0.52 mm to (147.3, 98.0)
- moved U3 0.48 mm to (124.5, 98.0)
- moved U9 0.42 mm to (147.3, 120.9)
- moved U8 0.36 mm to (124.5, 120.9)
- moved U12 0.34 mm to (147.3, 143.7)
- moved U6 0.31 mm to (147.3, 166.6)
- moved U11 0.27 mm to (124.5, 143.7)
- moved U4 0.23 mm to (124.5, 166.6)
Routing:
- net +3.3V: track 794.6 -> 782.4 mm
- net Net-(Q1-D): track 57.3 -> 59.3 mm
- net SDA: track 226.3 -> 225.0 mm
- net SCL: track 226.1 -> 224.9 mm
- net 1HZ_CLK: track 202.3 -> 201.8 mm
Other:
- board text added: "A"
- board text added: "B"

Commit message: Progress on station communications
Parts:
- J22: footprint easyeda2kicad:CONN-SMD_16P-P0.50_5034801600_1 -> easyeda2kicad:FPC-SMD_16P-P0.50_KH-FPC0.5-H1.0SMT-16P
- moved J22 0.05 mm to (146.1, 69.7)
- turned C17 to 0 degrees
- renumbered Boot to JP1, Solo to JP2
Connections:
- U7 pad 5: unconnected-(U7-WP-Pad5) -> GND
Routing:
- net +3.3V: track 782.4 -> 781.5 mm
- net Net-(C17-Pad1): track 5.10 -> 4.46 mm
