File: hardware/Apollo.kicad_pcb (KiCad board)
At the start: 2 copper layers, 101.2 x 199.1 mm, 80 parts, among them J1 TYPE-C 16PIN 2MD(073), J2 Conn_ARM_JTAG_SWD_10, J22 Conn_01x16, J3 Conn_02x03_Odd_Even, J4 Conn_02x04_Odd_Even, Q1 DMP1045U-7, Q2 SS8550, Q3 SS8050, Q4 SS8050, SW1 MK-12C01-G1.5, SW2 TS-1095PS-A1B2-C3D2, SW3 TS-1095PS-A1B2-C3D2, SW4 K1-1507SA-03, U1 TPS63031DSK, U10 PY25Q128HA, U11 SAINTCON-Minibadge, U12 SAINTCON-Minibadge, U2 RP2350A-QFN60, U3 SAINTCON-Minibadge, U4 SAINTCON-Minibadge, U5 SAINTCON-Minibadge, U6 SAINTCON-Minibadge, U7 24CS02, U8 SAINTCON-Minibadge, U9 SAINTCON-Minibadge, Y1 12Mhz

Commit message: Badge order placed. Hardware finalized
Parts:
- SW4: value K1-1507SA-03 -> LCK-TKLYABE0G1; footprint easyeda2kicad:KEY-SMD_K1-1507SA-03 -> easyeda2kicad:SW-SMD_10P-L10.6-W10.0_SKLYABE010
- U7: value 24CS02 -> 24CS08
- moved D7 0.80 mm to (168.9, 179.3)
- moved D6 0.79 mm to (123.1, 179.3)
- moved SW4 0.48 mm to (113.0, 172.2)
Connections:
- U2 pad 31: JOY_L -> JOY_R
- U2 pad 32: JOY_D -> JOY_B
- U2 pad 33: JOY_B -> JOY_D
- U2 pad 34: JOY_R -> JOY_L
Routing:
- net JOY_R: track 102.5 -> 97.3 mm
- net JOY_D: track 99.1 -> 103.8 mm
- net +3.3V: track 781.5 -> 778.0 mm
- net Net-(D6-DOUT): track 48.4 -> 49.9 mm
- net Net-(D5-DOUT): track 47.8 -> 48.8 mm
- net Net-(D7-DOUT): track 48.4 -> 49.3 mm
