File: hardware/i2c.kicad_sch (KiCad schematic)
At the start: 21 parts, among them Q2 SS8550, Q3 SS8050, U11 SAINTCON-Minibadge, U12 SAINTCON-Minibadge, U3 SAINTCON-Minibadge, U4 SAINTCON-Minibadge, U5 SAINTCON-Minibadge, U6 SAINTCON-Minibadge, U8 SAINTCON-Minibadge, U9 SAINTCON-Minibadge

Commit message: Badge order placed. Hardware finalized
Parts:
- R10, R11: LCSC Part C98220 -> C25804
Changed lines of the file:
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@@
 			)
 		)
-		(property "LCSC Part" "C98220"
+		(property "LCSC Part" "C25804"
 			(at 217.17 85.09 0)
 			(hide yes)
@@
 			)
 		)
-		(property "LCSC Part" "C98220"
+		(property "LCSC Part" "C25804"
 			(at 217.17 100.33 0)
 			(hide yes)
