File: hardware/mcu.kicad_sch (KiCad schematic)
At the start: 59 parts, among them J1 TYPE-C 16PIN 2MD(073), J2 Conn_ARM_JTAG_SWD_10, J22 Conn_01x16, J3 Conn_02x03_Odd_Even, J4 Conn_02x04_Odd_Even, Q1 DMP1045U-7, Q4 SS8050, SW1 MK-12C01-G1.5, SW2 TS-1095PS-A1B2-C3D2, SW3 TS-1095PS-A1B2-C3D2, SW4 K1-1507SA-03, U1 TPS63031DSK, U10 PY25Q128HA, U2 RP2350A-QFN60, U7 24CS02, Y1 12Mhz

Commit message: Badge order placed. Hardware finalized
Parts:
- removed SW4: K1-1507SA-03, easyeda2kicad:KEY-SMD_K1-1507SA-03, symbol easyeda2kicad:K1-1507SA-03
- added SW4: LCK-TKLYABE0G1, easyeda2kicad:SW-SMD_10P-L10.6-W10.0_SKLYABE010, symbol easyeda2kicad:LCK-TKLYABE0G1
- C10, C11, C12, C15, C4, C5, C6, C7, C8, C9: LCSC Part C14663 -> C1590
- C14: LCSC Part C19666 -> C1590
- L1: LCSC Part C395022 -> C167745
- R1: LCSC Part C14675 -> C25803
- R12: LCSC Part C98220 -> C25804
- R16: LCSC Part C108661 -> C23140
- R8, R9: LCSC Part C99782 -> C23162
- TP1, TP2, TP3: now left out of the parts list
- U7: value 24CS02 -> 24CS08; LCSC Part C18723540 -> C41408502
Connections:
- net GND: now also SW4.2, SW4.4, SW4.7, SW4.9
- net JOY_B: now also U2.32 (GPIO20), SW4.8; no longer U2.33 (GPIO21)
- net JOY_D: now also U2.33 (GPIO21), SW4.6; no longer U2.32 (GPIO20)
- net JOY_L: now also U2.34 (GPIO22), SW4.5; no longer U2.31 (GPIO19)
- net JOY_R: now also U2.31 (GPIO19), SW4.10; no longer U2.34 (GPIO22)
- net JOY_U: now also SW4.1
