File: hardware/Station/Station/Station.kicad_pcb (KiCad board)
At the start: 2 copper layers, 45 x 51.8 mm, 16 parts, among them J1 Conn_01x04, J2 Conn_01x04, J3 Conn_01x04, J4 Conn_01x04, J5 Conn_01x04, J6 Conn_01x03, J7 TYPE-C 16PIN 2MD(073)

Commit message: Station update before con
Parts:
- added C6: 10uF, Capacitor_SMD:C_0603_1608Metric_Pad1.08x0.95mm_HandSolder, F.Cu at (146.6, 98.8)
- added U1: M24C02-RMN, Package_SO:SOIC-8_3.9x4.9mm_P1.27mm, F.Cu at (146.3, 93.4)
Connections:
- A1 pad 31: unconnected-(A1-GPIO26_ADC0-Pad31) -> SDA
- A1 pad 32: unconnected-(A1-GPIO27_ADC1-Pad32) -> SCL
- A1 pad 36: unconnected-(A1-3V3-Pad36) -> +3V3
Routing:
- net +3V3: track 0.00 -> 21.9 mm
- net GND: track 23.6 -> 37.5 mm
- net SCL: track 0.00 -> 8.05 mm
- net SDA: track 0.00 -> 5.29 mm
- net Net-(A1-VSYS): track 17.2 -> 16.5 mm
